Commit message: adding missing links

File: hunter_pltf_description/description/depth_camera.urdf.xacro (robot description, xacro)
@@ -11,5 +11,5 @@
                     <origin xyz="0 0 0" rpy="1.57 0 1.57"/>
             <geometry>
-            <mesh filename="$(find hunter_pltf_description)/meshes/r200.dae">
+            <mesh filename="file://$(find hunter_pltf_description)/meshes/r200.dae">
             </mesh>
                 <!-- <box size="0.010 0.03 0.03"/> -->

File: hunter_pltf_description/description/hunter_pltf.urdf.xacro (robot description, xacro)
@@ -4,40 +4,20 @@
  <xacro:arg name="prefix" default="" />
  <xacro:if value="$(arg is_sim)">
-  <!--<xacro:include filename="$(find hunter_pltf_description)/description/depth_camera.urdf.xacro"/>-->
-  <xacro:include filename="$(find hunter_description)/description/hunter.urdf.xacro"/>
-  <!--<xacro:hunter_depth_camera name="back_camera" x="-1.2" y="-0.05" z="1.4" is_sim="$(arg is_sim)"/>-->
-  <!--<xacro:hunter_depth_camera name="front_camera" x="1.23" y="-0.05" z="1.4" is_sim="$(arg is_sim)"/>-->
+    <xacro:include filename="$(find hunter_description)/description/hunter.urdf.xacro"/>
  </xacro:if>
  <xacro:unless value="$(arg is_sim)">
   <xacro:include filename="$(find hunter_description)/description/hunter_core.urdf.xacro"/>
   <xacro:dogbot prefix="$(arg prefix)" is_sim="$(arg is_sim)"/>
-  <!-- <xacro:include filename="$(find hunter_description)/description/hunter_hardware.urdf.xacro"/> -->
-  <!-- <xacro:include filename="$(find hunter_pltf_description)/description/zed_multi.urdf.xacro"/> -->
-  <!-- <xacro:zed_depth_camera name="$(arg prefix)multi_link" x="0" y="0.0" z="0"/> -->
  </xacro:unless>
-    <!-- <link name="base_link" /> -->
     <xacro:include filename="$(find hunter_pltf_description)/description/lidar.urdf.xacro"/>
     <xacro:include filename="$(find hunter_pltf_description)/description/mid360.xacro"/>
     <xacro:include filename="$(find hunter_pltf_description)/description/imu.urdf.xacro"/>
     <xacro:include filename="$(find hunter_pltf_description)/description/gps.urdf.xacro"/>
-    <!--  ADD ADDITIONAL SENSOR URDF HERE   -->
-    <!--  -->
-<!-- <xacro:include filename="$(find hunter_pltf_description)/description/depth_camera.urdf.xacro"/> -->
-    <xacro:hunter_imu name="$(arg prefix)imu1" is_sim="$(arg is_sim)" x="-0.40" y="0.0" z="0.596"/>
-    <xacro:hunter_imu name="$(arg prefix)imu2" is_sim="$(arg is_sim)" x="1.2" y="0.0" z="0.4" />
-    <!-- <xacro:mid360 name="$(arg prefix)front_lidar" xyz="1.2 0.3 0.3" rpy="0 0 0"/> -->
-    <!-- <xacro:mid360 name="$(arg prefix)back_lidar" xyz="-1.2 -0.3 0.3" rpy="0 0 0"/> -->
-    <!-- <xacro:hunter_lidar name="$(arg prefix)front_lidar" x="1.2" y="0.3" z="0.3"/> -->
-    <!-- <xacro:hunter_lidar name="$(arg prefix)back_lidar" x="-1.2" y="-0.3" z="0.3"/> -->
-    <!-- <xacro:hunter_depth_camera name="$(arg prefix)back_camera" x="-1.2" y="0.0" z="0.6" yaw='3.14' is_sim="$(arg is_sim)"/> -->
-    <!-- <xacro:hunter_depth_camera name="$(arg prefix)front_camera" x="1.2" y="0.0" z="0.6" is_sim="$(arg is_sim)"/> -->
-    <xacro:hunter_gps name="$(arg prefix)gps_base" is_sim="$(arg is_sim)" x="-0.40" y="0.0" z="0.616"/>
-    <xacro:hunter_gps name="$(arg prefix)gps_rover" is_sim="$(arg is_sim)" x="-0.40" y="0.0" z="0.616"/>
-        <!-- Lidar -->
-    <!-- <xacro:mid360 name="livox_front" parent="base_link" topic="front_lidar/scan">
-      <origin xyz="1.05 0.35 0.37" rpy="0 0 3.14"/>
-    </xacro:mid360> -->
-    <!-- <xacro:mid360 name="livox_back" parent="base_link" topic="back_lidar/scan">
-      <origin xyz="-1.05 -0.35 0.37" rpy="0 0 0"/>
-    </xacro:mid360> -->
+    <xacro:include filename="$(find hunter_pltf_description)/description/depth_camera.urdf.xacro"/>
+    <xacro:hunter_imu name="$(arg prefix)imu1" is_sim="$(arg is_sim)" x="0.0" y="0.0" z="0.2"/>
+    <xacro:hunter_lidar name="$(arg prefix)front_lidar" x="0.4" y="-0.2" z="0.37"/>
+    <xacro:hunter_lidar name="$(arg prefix)back_lidar" x="-0.4" y="0.2" z="0.37"  yaw="3.14"/>
+    <xacro:hunter_depth_camera name="front_camera" x="0.3" y="-0.05" z="1.4" is_sim="$(arg is_sim)" />
+    <xacro:hunter_depth_camera name="back_camera" x="-0.3" y="-0.05" z="1.4" is_sim="$(arg is_sim)" yaw="3.14"/>
+    <xacro:hunter_gps name="$(arg prefix)gps_base" is_sim="$(arg is_sim)" x="-0.0" y="0.0" z="0.2"/>
 </robot>

Commit message: Refactor + add zed2 model

File: hunter_pltf_description/description/depth_camera.urdf.xacro (robot description, xacro)
@@ -9,11 +9,8 @@
     <link name="${name}_link">
         <visual>
-                    <origin xyz="0 0 0" rpy="1.57 0 1.57"/>
+            <origin xyz="0 0 0" rpy="0 0 -1.57"/>
             <geometry>
-            <mesh filename="file://$(find hunter_pltf_description)/meshes/r200.dae">
-            </mesh>
-                <!-- <box size="0.010 0.03 0.03"/> -->
+                <mesh filename="file://$(find hunter_pltf_description)/meshes/zed2.dae"/>
             </geometry>
-            <!-- <material name="red"/> -->
         </visual>
     </link>
@@ -26,5 +23,4 @@
 <xacro:if value="${is_sim}">
     <gazebo reference="${name}_link">
-        <!-- <material>Gazebo/Red</material> -->
         <sensor name="${name}_camera" type="depth">
             <pose> 0 0 0 0 0 0 </pose>

File: hunter_pltf_description/description/hunter_pltf.urdf.xacro (robot description, xacro)
@@ -4,9 +4,8 @@
    <xacro:arg name="prefix" default="" />
    <xacro:if value="$(arg is_sim)">
-      <xacro:include filename="$(find hunter_description)/description/hunter.urdf.xacro"/>
+      <xacro:include filename="$(find hunter_description)/description/robot.urdf.xacro"/>
    </xacro:if>
    <xacro:unless value="$(arg is_sim)">
-   <xacro:include filename="$(find hunter_description)/description/hunter_core.urdf.xacro"/>
-   <xacro:dogbot prefix="$(arg prefix)" is_sim="$(arg is_sim)"/>
+   <xacro:include filename="$(find hunter_description)/description/robot_core.xacro"/>
    </xacro:unless>
    <xacro:include filename="$(find hunter_pltf_description)/description/lidar.urdf.xacro"/>
@@ -18,10 +17,10 @@
    <xacro:hunter_lidar name="$(arg prefix)front_lidar" x="0.615" y="0.28" z="0.33" is_sim="$(arg is_sim)" />
    <xacro:hunter_lidar name="$(arg prefix)back_lidar" x="-0.565" y="-0.28" z="0.33"  yaw="3.14" is_sim="$(arg is_sim)"/>
-   <xacro:hunter_depth_camera name="front_camera" x="0.55" y="-0.00" z="0.61" is_sim="$(arg is_sim)" />
-   <xacro:hunter_depth_camera name="back_camera" x="-0.55" y="-0.00" z="0.61" is_sim="$(arg is_sim)" yaw="3.14"/>
-   <xacro:hunter_depth_camera name="fish_front_camera" x="0.55" y="0.00" z="0.93" is_sim="$(arg is_sim)" />
-   <xacro:hunter_depth_camera name="fish_right_camera" x="0.495" y="0.08" z="0.93" is_sim="$(arg is_sim)"  yaw="1.57"/>
+   <xacro:hunter_depth_camera name="front_camera" x="0.55" y="-0.00" z="0.50" is_sim="$(arg is_sim)" />
+   <xacro:hunter_depth_camera name="back_camera" x="-0.55" y="-0.00" z="0.50" is_sim="$(arg is_sim)" yaw="3.14"/>
+   <!-- <xacro:hunter_depth_camera name="fish_front_camera" x="0.55" y="0.00" z="0.93" is_sim="$(arg is_sim)" />
+   <xacro:hunter_depth_camera name="fish_right_camera" x="0.495" y="0.08" z="0.93" is_sim="$(arg is_sim)"  yaw="1.57"/> -->
    <!-- <xacro:hunter_depth_camera name="fish_back_camera" x="0.179" y="0.00" z="1.28" is_sim="$(arg is_sim)" yaw="3.14" />-->
-   <xacro:hunter_depth_camera name="fish_left_camera" x="0.495" y="-0.08" z="0.93" is_sim="$(arg is_sim)" yaw="-1.57" />
+   <!-- <xacro:hunter_depth_camera name="fish_left_camera" x="0.495" y="-0.08" z="0.93" is_sim="$(arg is_sim)" yaw="-1.57" /> -->
    <xacro:hunter_gps name="$(arg prefix)gps_base" is_sim="$(arg is_sim)" x="-0.25" y="0.0" z="0.33"/>
    <xacro:hunter_gps name="$(arg prefix)back_antenna" is_sim="$(arg is_sim)" x="-0.5" y="-0.245" z="0.80"/>

File: hunter_pltf_description/description/imu.urdf.xacro (robot description, xacro)
@@ -1,27 +1,48 @@
 <?xml version="1.0"?>
-<robot xmlns:xacro="http://www.ros.org/wiki/xacro" >
- <xacro:macro name="hunter_imu" params="name topic x:=0.0 y:=0.0 z:=0.0 roll:=0.0 pitch:=0.0 yaw:=0.0 is_sim:=true">
-  <joint name="${name}_joint" type='fixed'>
-   <parent link="base_link"/>
-   <child link="${name}_link"/>
-   <origin xyz="${x} ${y} ${z}" rpy="${roll} ${pitch} ${yaw}"/>
-  </joint>
-  <link name="${name}_link"/>
- <xacro:if value="${is_sim}">
-    <gazebo reference="${name}_link">
-      <sensor name="${name}_imu" type="imu">
-      <plugin filename="libgazebo_ros_imu_sensor.so" name="${name}_controller">
-          <ros>
-            <!-- <namespace>$(arg prefix)</namespace> -->
-            <remapping>~/out:=${topic}</remapping>
-            <initial_orientation_as_reference>false</initial_orientation_as_reference>
-          </ros>
-          <frame_name>${name}_link</frame_name>
-        </plugin>
-        <always_on>true</always_on>
-        <update_rate>10</update_rate>
-      </sensor>
-    </gazebo>
- </xacro:if>
-</xacro:macro>
+<robot xmlns:xacro="http://www.ros.org/wiki/xacro">
+  <xacro:macro name="hunter_imu" params="name topic x:=0.0 y:=0.0 z:=0.0 roll:=0.0 pitch:=0.0 yaw:=0.0 is_sim:=true">
+    <joint name="${name}_joint" type="fixed">
+      <parent link="base_link"/>
+      <child link="${name}_link"/>
+      <origin xyz="${x} ${y} ${z}" rpy="${roll} ${pitch} ${yaw}"/>
+    </joint>
+    <link name="${name}_link"/>
+    <xacro:if value="${is_sim}">
+      <gazebo reference="${name}_link">
+        <sensor name="${name}_imu" type="imu">
+          <plugin filename="libgazebo_ros_imu_sensor.so" name="${name}_controller">
+            <ros>
+              <remapping>~/out:=${topic}</remapping>
+              <initial_orientation_as_reference>false</initial_orientation_as_reference>
+            </ros>
+            <frame_name>${name}_link</frame_name>
+          </plugin>
+          <always_on>true</always_on>
+          <update_rate>50</update_rate>
+          <imu>
+            <angular_velocity>
+              <noise type="gaussian">
+                <mean>0.0</mean>
+                <stddev>0.01</stddev>
+              </noise>
+              <bias>
+                <mean>0.0</mean>
+                <stddev>0.0001</stddev>
+              </bias>
+            </angular_velocity>
+            <linear_acceleration>
+              <noise type="gaussian">
+                <mean>0.0</mean>
+                <stddev>0.01</stddev>
+              </noise>
+              <bias>
+                <mean>0.0</mean>
+                <stddev>0.0001</stddev>
+              </bias>
+            </linear_acceleration>
+          </imu>
+        </sensor>
+      </gazebo>
+    </xacro:if>
+  </xacro:macro>
 </robot>

File: hunter_pltf_description/description/lidar.urdf.xacro (robot description, xacro)
@@ -19,5 +19,7 @@
                 <cylinder radius="0.01" length="0.1"/>
             </geometry>
-            <material name="black"/>
+            <material name="black">
+                <color rgba="0 0 0 1"/>
+            </material>
         </visual>
         <collision>
