Commit message: updated livox xacro

File: hunter_pltf_description/description/mid360.xacro (robot description, xacro)
@@ -3,80 +3,84 @@
   <xacro:property name="M_PI" value="3.1415926"/>
   <xacro:property name="laser_min_range" value="0.1"/>
-  <xacro:property name="laser_max_range" value="200.0"/>
+  <xacro:property name="laser_max_range" value="100.0"/>
   <xacro:property name="samples" value="10000"/>
   <xacro:property name="resolution" value="0.002"/>
   <xacro:property name="noise_mean" value="0.0"/>
   <xacro:property name="noise_stddev" value="0.01"/>
-  <xacro:property name="is_sim" value="true"/>
-  <xacro:property name="mass" value="0.4" />
-  <xacro:property name="length" value="0.1" />
-  <xacro:property name="width" value="0.06" />
-  <xacro:property name="height" value="0.06" />
+  <xacro:property name="mass" value="0.4"/>
+  <xacro:property name="length" value="0.1"/>
+  <xacro:property name="width" value="0.06"/>
+  <xacro:property name="height" value="0.06"/>
+  <!-- Macro to calculate box inertia -->
   <xacro:macro name="box_inertia" params="m w h d">
     <inertial>
-      <origin xyz="0 0 0" rpy="${pi/2} 0 ${pi/2}"/>
+      <origin xyz="0 0 0" rpy="0 0 0"/>
       <mass value="${m}"/>
-      <inertia ixx="${(m/12) * (h*h + d*d)}" ixy="0.0" ixz="0.0" iyy="${(m/12) * (w*w + d*d)}" iyz="0.0" izz="${(m/12) * (w*w + h*h)}"/>
+      <inertia ixx="${m/12 * (h*h + d*d)}"
+               ixy="0.0"
+               ixz="0.0"
+               iyy="${m/12 * (w*w + d*d)}"
+               iyz="0.0"
+               izz="${m/12 * (w*w + h*h)}"/>
     </inertial>
   </xacro:macro>
-  <xacro:macro name="mid360" params="name:='' parent:= 'base_link' topic:='mid360' *origin ">
-<link name="${name}">
-<xacro:box_inertia m="${length}" w="${width}" d="${length}" h="${height}"/>
-  <visual>
-        <!-- <geometry>
-            <box size="${length} ${width} ${height}"/>
-        </geometry> -->
+  <!-- Macro to define the mid360 lidar sensor -->
+  <xacro:macro name="mid360" params="name='' parent='base_link' topic='mid360' origin_xyz='0 0 0' origin_rpy='0 0 0' is_sim:=true">
+    <link name="${name}">
+      <xacro:box_inertia m="${mass}" w="${width}" d="${length}" h="${height}"/>
+      <visual>
         <geometry>
-          <mesh filename="$(find ros2_livox_simulation)/meshes/mid-360-scaled.dae">
-          </mesh>
+          <mesh filename="$(find ros2_livox_simulation)/meshes/mid-360-scaled.dae"/>
         </geometry>
-  </visual>
-</link>
+      </visual>
+    </link>
     <joint name="${name}_joint" type="fixed">
       <parent link="${parent}"/>
       <child link="${name}"/>
-      <xacro:insert_block name="origin"/>
+      <origin xyz="${origin_xyz}" rpy="${origin_rpy}"/>
     </joint>
-    <gazebo reference="${name}">
-      <sensor type="ray" name="${name}">
-        <pose>0 0 0 0 0 0</pose>
-        <visualize>true</visualize>
-        <update_rate>10</update_rate>
-        <!-- This ray plgin is only for visualization. -->
-        <plugin name="${name}_plugin" filename="libros2_livox.so">
-			<ray>
-			  <scan>
-				<horizontal>
-				<samples>100</samples>
-				<resolution>1</resolution>
-				<min_angle>${0}</min_angle>
-				<max_angle>${2*M_PI}</max_angle>
-				</horizontal>
-				<vertical>
-				<samples>360</samples>
-				<resolution>1</resolution>
-				<min_angle>${-7.22/180*M_PI}</min_angle>
-				<max_angle>${55.22/180*M_PI}</max_angle>
-				</vertical>
-			  </scan>
-			  <range>
-				<min>${laser_min_range}</min>
-				<max>${laser_max_range}</max>
-				<resolution>${resolution}</resolution>
-			  </range>
-			  <noise>
-				<type>gaussian</type>
-				<mean>${noise_mean}</mean>
-				<stddev>${noise_stddev}</stddev>
-			  </noise>
-			</ray>
-          <visualize>false</visualize>
-		  <samples>${samples}</samples>
-		  <downsample>1</downsample>
-		  <csv_file_name>$(find ros2_livox_simulation)/scan_mode/mid360.csv</csv_file_name>
-		  <topic>${topic}</topic>
-        </plugin>
-      </sensor>
-    </gazebo>
+    <xacro:if value="${is_sim}">
+      <gazebo reference="${name}">
+        <sensor type="ray" name="${name}">
+          <!-- <pose>${origin_xyz} ${origin_rpy}</pose> -->
+          <pose>0 0 0 0 0 0</pose>
+          <visualize>true</visualize>
+          <update_rate>10</update_rate>
+          <plugin name="${name}_plugin" filename="libros2_livox.so">
+            <ray>
+              <scan>
+                <horizontal>
+                  <samples>100</samples>
+                  <resolution>1</resolution>
+                  <min_angle>0</min_angle>
+                  <max_angle>${2 * M_PI}</max_angle>
+                </horizontal>
+                <vertical>
+                  <samples>360</samples>
+                  <resolution>1</resolution>
+                  <min_angle>${-7.22 / 180 * M_PI}</min_angle>
+                  <max_angle>${55.22 / 180 * M_PI}</max_angle>
+                </vertical>
+              </scan>
+              <range>
+                <min>${laser_min_range}</min>
+                <max>${laser_max_range}</max>
+                <resolution>${resolution}</resolution>
+              </range>
+              <noise>
+                <type>gaussian</type>
+                <mean>${noise_mean}</mean>
+                <stddev>${noise_stddev}</stddev>
+              </noise>
+            </ray>
+            <visualize>false</visualize>
+            <samples>${samples}</samples>
+            <downsample>5</downsample>
+            <csv_file_name>$(find ros2_livox_simulation)/scan_mode/mid360.csv</csv_file_name>
+            <topic>${topic}</topic>
+          </plugin>
+        </sensor>
+      </gazebo>
+    </xacro:if>
   </xacro:macro>
 </robot>

Commit message: fix livox urdf

File: hunter_pltf_description/description/mid360.xacro (robot description, xacro)
@@ -31,7 +31,12 @@
       <visual>
         <geometry>
-          <mesh filename="$(find ros2_livox_simulation)/meshes/mid-360-scaled.dae"/>
+          <mesh filename="file://$(find hunter_pltf_description)/meshes/livox360.dae"/>
         </geometry>
       </visual>
+      <collision>
+        <geometry>
+          <mesh filename="file://$(find hunter_pltf_description)/meshes/livox360.dae"/>
+        </geometry>
+      </collision>
     </link>
     <joint name="${name}_joint" type="fixed">
@@ -76,5 +81,5 @@
             <visualize>false</visualize>
             <samples>${samples}</samples>
-            <downsample>5</downsample>
+            <downsample>1</downsample>
             <csv_file_name>$(find ros2_livox_simulation)/scan_mode/mid360.csv</csv_file_name>
             <topic>${topic}</topic>
