Commit message: Update mid360.xacro to enhance lidar sensor configuration and increase sample count

File: hunter_pltf_description/description/mid360.xacro (robot description, xacro)
@@ -4,5 +4,5 @@
   <xacro:property name="laser_min_range" value="0.1"/>
   <xacro:property name="laser_max_range" value="100.0"/>
-  <xacro:property name="samples" value="10000"/>
+  <xacro:property name="samples" value="24000"/>
   <xacro:property name="resolution" value="0.002"/>
   <xacro:property name="noise_mean" value="0.0"/>
@@ -26,15 +26,22 @@
   </xacro:macro>
   <!-- Macro to define the mid360 lidar sensor -->
-  <xacro:macro name="mid360" params="name='' parent='base_link' topic='mid360' origin_xyz='0 0 0' origin_rpy='0 0 0' is_sim:=true">
+  <xacro:macro name="mid360"
+               params="name='' parent='base_link'
+                       raw_topic:='mid360/raw_gpu'
+                       topic:='mid360/points'
+                       diagnostics_topic:='mid360/diagnostics'
+                       frame_id:=''
+                       origin_xyz='0 0 0' origin_rpy='0 0 0'
+                       is_sim:=true">
     <link name="${name}">
       <xacro:box_inertia m="${mass}" w="${width}" d="${length}" h="${height}"/>
       <visual>
         <geometry>
-          <mesh filename="file://$(find hunter_pltf_description)/meshes/livox360.dae"/>
+          <mesh filename="package://hunter_pltf_description/meshes/livox360.dae"/>
         </geometry>
       </visual>
       <collision>
         <geometry>
-          <mesh filename="file://$(find hunter_pltf_description)/meshes/livox360.dae"/>
+          <mesh filename="package://hunter_pltf_description/meshes/livox360.dae"/>
         </geometry>
       </collision>
@@ -47,43 +54,53 @@
     <xacro:if value="${is_sim}">
       <gazebo reference="${name}">
-        <sensor type="ray" name="${name}">
-          <!-- <pose>${origin_xyz} ${origin_rpy}</pose> -->
+        <sensor type="gpu_lidar" name="${name}_raw_gpu_lidar">
+          <topic>${raw_topic}</topic>
+          <gz_frame_id>${frame_id}</gz_frame_id>
           <pose>0 0 0 0 0 0</pose>
           <visualize>true</visualize>
           <update_rate>10</update_rate>
-          <plugin name="${name}_plugin" filename="libros2_livox.so">
-            <ray>
-              <scan>
-                <horizontal>
-                  <samples>100</samples>
-                  <resolution>1</resolution>
-                  <min_angle>0</min_angle>
-                  <max_angle>${2 * M_PI}</max_angle>
-                </horizontal>
-                <vertical>
-                  <samples>360</samples>
-                  <resolution>1</resolution>
-                  <min_angle>${-7.22 / 180 * M_PI}</min_angle>
-                  <max_angle>${55.22 / 180 * M_PI}</max_angle>
-                </vertical>
-              </scan>
-              <range>
-                <min>${laser_min_range}</min>
-                <max>${laser_max_range}</max>
-                <resolution>${resolution}</resolution>
-              </range>
-              <noise>
-                <type>gaussian</type>
-                <mean>${noise_mean}</mean>
-                <stddev>${noise_stddev}</stddev>
-              </noise>
-            </ray>
-            <visualize>false</visualize>
-            <samples>${samples}</samples>
-            <downsample>5</downsample>
-            <csv_file_name>$(find livox_mid360_gz)/scan_mode/mid360.csv</csv_file_name>
-            <topic>${topic}</topic>
-          </plugin>
+          <lidar>
+            <scan>
+              <horizontal>
+                <samples>1024</samples>
+                <resolution>1</resolution>
+                <min_angle>${-M_PI}</min_angle>
+                <max_angle>${M_PI}</max_angle>
+              </horizontal>
+              <vertical>
+                <samples>256</samples>
+                <resolution>1</resolution>
+                <min_angle>${-7.22 / 180 * M_PI}</min_angle>
+                <max_angle>${55.22 / 180 * M_PI}</max_angle>
+              </vertical>
+            </scan>
+            <range>
+              <min>${laser_min_range}</min>
+              <max>${laser_max_range}</max>
+              <resolution>${resolution}</resolution>
+            </range>
+          </lidar>
         </sensor>
+      </gazebo>
+      <gazebo>
+        <plugin filename="liblivox_mid360_gz_plugin.so"
+                name="livox_mid360_gz::LivoxMid360GpuLidar">
+          <input_topic>${raw_topic}/points</input_topic>
+          <output_topic>${topic}</output_topic>
+          <diagnostics_topic>${diagnostics_topic}</diagnostics_topic>
+          <frame_id>${frame_id}</frame_id>
+          <frame_rate>10</frame_rate>
+          <samples>${samples}</samples>
+          <downsample>5</downsample>
+          <scan_pattern_file>package://livox_mid360_gz/scan_mode/mid360.csv</scan_pattern_file>
+          <min_range>${laser_min_range}</min_range>
+          <max_range>${laser_max_range}</max_range>
+          <range_noise_stddev>${noise_stddev}</range_noise_stddev>
+          <angular_noise_stddev>0.0</angular_noise_stddev>
+          <input_horizontal_samples>1024</input_horizontal_samples>
+          <input_vertical_samples>256</input_vertical_samples>
+          <input_min_elevation>${-7.22 / 180 * M_PI}</input_min_elevation>
+          <input_max_elevation>${55.22 / 180 * M_PI}</input_max_elevation>
+        </plugin>
       </gazebo>
     </xacro:if>
