Commit message: Update GPS URDF configuration and adjust downsample rate in mid360.xacro

File: hunter_pltf_description/description/gps.urdf.xacro (robot description, xacro)
@@ -1,26 +1,30 @@
 <?xml version="1.0"?>
-<robot xmlns:xacro="http://www.ros.org/wiki/xacro" >
- <xacro:macro name="hunter_gps" params="name x:=0.0 y:=0.0 z:=0.0 roll:=0.0 pitch:=0.0 yaw:=0.0 is_sim:=true">
-  <joint name="${name}_joint" type='fixed'>
-   <parent link="base_link"/>
-   <child link="${name}_link"/>
-   <origin xyz="${x} ${y} ${z}" rpy="${roll} ${pitch} ${yaw}"/>
-  </joint>
-  <link name="${name}_link"/>
- <xacro:if value="${is_sim}">
-    <gazebo reference="${name}_link">
-      <sensor name="${name}_gps" type="gps">
-      <plugin filename="libgazebo_ros_gps_sensor.so" name="${name}_controller">
-          <ros>
-            <!-- <namespace>$(arg prefix)</namespace> -->
-            <remapping>~/out:=/${name}/fix</remapping>
-          </ros>
-          <frame_name>${name}_link</frame_name>
-        </plugin>
-        <always_on>true</always_on>
-        <update_rate>10</update_rate>
-      </sensor>
-    </gazebo>
- </xacro:if>
-</xacro:macro>
+<robot xmlns:xacro="http://www.ros.org/wiki/xacro">
+  <xacro:macro name="hunter_gps" params="name x:=0.0 y:=0.0 z:=0.0 roll:=0.0 pitch:=0.0 yaw:=0.0 is_sim:=true">
+    <!-- Choose yaw value: force to 0.0 in simulation, else use provided yaw -->
+    <xacro:property name="final_yaw" value="${0.0 if is_sim else yaw}" />
+    <!-- Define the joint and link once -->
+    <joint name="${name}_joint" type="fixed">
+      <parent link="base_link"/>
+      <child link="${name}_link"/>
+      <origin xyz="${x} ${y} ${z}" rpy="${roll} ${pitch} ${final_yaw}"/>
+    </joint>
+    <link name="${name}_link"/>
+    <!-- Add Gazebo sensor only when in simulation -->
+    <xacro:if value="${is_sim}">
+      <gazebo reference="${name}_link">
+        <sensor name="${name}_gps" type="gps">
+          <plugin filename="libgazebo_ros_gps_sensor.so" name="${name}_controller">
+            <ros>
+              <!-- <namespace>$(arg prefix)</namespace> -->
+              <remapping>~/out:=/${name}/fix</remapping>
+            </ros>
+            <frame_name>${name}_link</frame_name>
+          </plugin>
+          <always_on>true</always_on>
+          <update_rate>10</update_rate>
+        </sensor>
+      </gazebo>
+    </xacro:if>
+  </xacro:macro>
 </robot>

File: hunter_pltf_description/description/hunter_pltf.urdf.xacro (robot description, xacro)
@@ -23,5 +23,5 @@
    <!-- <xacro:hunter_depth_camera name="fish_back_camera" x="0.179" y="0.00" z="1.28" is_sim="$(arg is_sim)" yaw="3.14" />-->
    <!-- <xacro:hunter_depth_camera name="fish_left_camera" x="0.495" y="-0.08" z="0.93" is_sim="$(arg is_sim)" yaw="-1.57" /> -->
-   <xacro:hunter_gps name="$(arg prefix)gps_base" is_sim="$(arg is_sim)" x="-0.25" y="0.0" z="0.33"/>
+   <xacro:hunter_gps name="$(arg prefix)gps_base" is_sim="$(arg is_sim)" x="-0.25" y="0.0" z="0.33" yaw="0.037482" />
    <!-- <xacro:hunter_gps name="$(arg prefix)back_antenna" is_sim="$(arg is_sim)" x="-0.5" y="-0.245" z="0.80"/> -->
    <!-- <xacro:hunter_gps name="$(arg prefix)front_antenna" is_sim="$(arg is_sim)" x="0.5" y="-0.245" z="0.80"/> -->

File: hunter_pltf_description/description/mid360.xacro (robot description, xacro)
@@ -81,5 +81,5 @@
             <visualize>false</visualize>
             <samples>${samples}</samples>
-            <downsample>1</downsample>
+            <downsample>10</downsample>
             <csv_file_name>$(find ros2_livox_simulation)/scan_mode/mid360.csv</csv_file_name>
             <topic>${topic}</topic>
