Commit message: tf fix and real robot launch

File: hunter_pltf_description/description/hunter_pltf.urdf.xacro (robot description, xacro)
@@ -10,8 +10,11 @@
  </xacro:if>
  <xacro:unless value="$(arg is_sim)">
-  <xacro:include filename="$(find hunter_description)/description/hunter_hardware.urdf.xacro"/>
-  <xacro:include filename="$(find hunter_pltf_description)/description/zed_multi.urdf.xacro"/>
-  <xacro:zed_depth_camera name="$(arg prefix)multi_link" x="0" y="0.0" z="0"/>
+  <xacro:include filename="$(find hunter_description)/description/hunter_core.urdf.xacro"/>
+  <xacro:dogbot prefix="$(arg prefix)" is_sim="$(arg is_sim)"/>
+  <!-- <xacro:include filename="$(find hunter_description)/description/hunter_hardware.urdf.xacro"/> -->
+  <!-- <xacro:include filename="$(find hunter_pltf_description)/description/zed_multi.urdf.xacro"/> -->
+  <!-- <xacro:zed_depth_camera name="$(arg prefix)multi_link" x="0" y="0.0" z="0"/> -->
  </xacro:unless>
+    <!-- <link name="base_link" /> -->
     <xacro:include filename="$(find hunter_pltf_description)/description/lidar.urdf.xacro"/>
     <xacro:include filename="$(find hunter_pltf_description)/description/mid360.xacro"/>

Commit message: adding topic for imu sensor

File: hunter_pltf_description/description/hunter_pltf.urdf.xacro (robot description, xacro)
@@ -15,5 +15,5 @@
     <xacro:include filename="$(find hunter_pltf_description)/description/gps.urdf.xacro"/>
     <xacro:include filename="$(find hunter_pltf_description)/description/depth_camera.urdf.xacro"/>
-    <xacro:hunter_imu name="$(arg prefix)imu1" is_sim="$(arg is_sim)" x="0.0" y="0.0" z="0.2"/>
+    <xacro:hunter_imu name="$(arg prefix)imu1" is_sim="$(arg is_sim)" x="0.0" y="0.0" z="0.2" topic="/gps_base/yaw"/>
     <xacro:hunter_lidar name="$(arg prefix)front_lidar" x="0.4" y="-0.2" z="0.37"/>
     <xacro:hunter_lidar name="$(arg prefix)back_lidar" x="-0.4" y="0.2" z="0.37"  yaw="3.14"/>

File: hunter_pltf_description/description/imu.urdf.xacro (robot description, xacro)
@@ -1,5 +1,5 @@
 <?xml version="1.0"?>
 <robot xmlns:xacro="http://www.ros.org/wiki/xacro" >
- <xacro:macro name="hunter_imu" params="name x:=0.0 y:=0.0 z:=0.0 roll:=0.0 pitch:=0.0 yaw:=0.0 is_sim:=true">
+ <xacro:macro name="hunter_imu" params="name topic x:=0.0 y:=0.0 z:=0.0 roll:=0.0 pitch:=0.0 yaw:=0.0 is_sim:=true">
   <joint name="${name}_joint" type='fixed'>
    <parent link="base_link"/>
@@ -14,5 +14,5 @@
           <ros>
             <!-- <namespace>$(arg prefix)</namespace> -->
-            <remapping>~/out:=/${name}/data</remapping>
+            <remapping>~/out:=${topic}</remapping>
             <initial_orientation_as_reference>false</initial_orientation_as_reference>
           </ros>

Commit message: Update lidar properties and adjust downsample rate in mid360 configuration

File: hunter_pltf_description/description/hunter_pltf.urdf.xacro (robot description, xacro)
@@ -5,7 +5,11 @@
    <xacro:if value="$(arg is_sim)">
       <xacro:include filename="$(find hunter_description)/description/robot.urdf.xacro"/>
+      <xacro:property name="front_lidar_rpy" value="0 0 0"/>
+      <xacro:property name="back_lidar_rpy" value="0 0 3.14159"/>
    </xacro:if>
    <xacro:unless value="$(arg is_sim)">
-   <xacro:include filename="$(find hunter_description)/description/robot_core_real_hack.xacro"/>
+      <xacro:include filename="$(find hunter_description)/description/robot_core_real_hack.xacro"/>
+      <xacro:property name="front_lidar_rpy" value="0 0 -0.0261799"/>
+      <xacro:property name="back_lidar_rpy" value="-0.174533 0 3.14159"/>
    </xacro:unless>
    <xacro:include filename="$(find hunter_pltf_description)/description/lidar.urdf.xacro"/>
@@ -14,5 +18,5 @@
    <xacro:include filename="$(find hunter_pltf_description)/description/gps.urdf.xacro"/>
    <xacro:include filename="$(find hunter_pltf_description)/description/depth_camera.urdf.xacro"/>
-   <xacro:hunter_imu name="$(arg prefix)imu1" is_sim="$(arg is_sim)" x="0.0" y="0.0" z="0.2" topic="/gps_base/yaw"/>
+   <xacro:hunter_imu name="$(arg prefix)imu" is_sim="$(arg is_sim)" x="0.0" y="0.0" z="0.2" topic="/imu/data"/>
    <!-- <xacro:hunter_lidar name="$(arg prefix)front_lidar" x="0.615" y="0.28" z="0.33" is_sim="$(arg is_sim)" /> -->
    <!-- <xacro:hunter_lidar name="$(arg prefix)back_lidar" x="-0.565" y="-0.28" z="0.33"  yaw="3.14" is_sim="$(arg is_sim)"/> -->
@@ -26,5 +30,5 @@
    <!-- <xacro:hunter_gps name="$(arg prefix)back_antenna" is_sim="$(arg is_sim)" x="-0.5" y="-0.245" z="0.80"/> -->
    <!-- <xacro:hunter_gps name="$(arg prefix)front_antenna" is_sim="$(arg is_sim)" x="0.5" y="-0.245" z="0.80"/> -->
-   <xacro:mid360 name="$(arg prefix)front_lidar_link" topic="front_lidar/points" origin_xyz="0.615 0.28 0.33" origin_rpy="0 0 -0.0261799" is_sim="$(arg is_sim)"/>
-   <xacro:mid360 name="$(arg prefix)back_lidar_link" topic="back_lidar/points" origin_xyz="-0.615 -0.28 0.33" origin_rpy="-0.174533 0 3.14159" is_sim="$(arg is_sim)"/>
+   <xacro:mid360 name="$(arg prefix)front_lidar_link" topic="front_lidar/points" origin_xyz="0.615 0.28 0.33" origin_rpy="${front_lidar_rpy}" is_sim="$(arg is_sim)"/>
+   <xacro:mid360 name="$(arg prefix)back_lidar_link" topic="back_lidar/points" origin_xyz="-0.615 -0.28 0.33" origin_rpy="${back_lidar_rpy}" is_sim="$(arg is_sim)"/>
 </robot>

File: hunter_pltf_description/description/mid360.xacro (robot description, xacro)
@@ -81,5 +81,5 @@
             <visualize>false</visualize>
             <samples>${samples}</samples>
-            <downsample>10</downsample>
+            <downsample>5</downsample>
             <csv_file_name>$(find ros2_livox_simulation)/scan_mode/mid360.csv</csv_file_name>
             <topic>${topic}</topic>

Commit message: fix urdf

File: hunter_pltf_description/description/hunter_pltf.urdf.xacro (robot description, xacro)
@@ -10,6 +10,6 @@
    <xacro:unless value="$(arg is_sim)">
       <xacro:include filename="$(find hunter_description)/description/robot_core_real_hack.xacro"/>
-      <xacro:property name="front_lidar_rpy" value="0 0 -0.0261799"/>
-      <xacro:property name="back_lidar_rpy" value="-0.174533 0 3.14159"/>
+      <xacro:property name="front_lidar_rpy" value="0 0 0"/>
+      <xacro:property name="back_lidar_rpy" value="0 0 3.14159"/>
    </xacro:unless>
    <xacro:include filename="$(find hunter_pltf_description)/description/lidar.urdf.xacro"/>
@@ -18,18 +18,18 @@
    <xacro:include filename="$(find hunter_pltf_description)/description/gps.urdf.xacro"/>
    <xacro:include filename="$(find hunter_pltf_description)/description/depth_camera.urdf.xacro"/>
-   <xacro:hunter_imu name="$(arg prefix)imu" is_sim="$(arg is_sim)" x="-0.25" y="0.0" z="0.33" topic="/gps_base/yaw"/>
-   <xacro:hunter_imu name="$(arg prefix)imu1" is_sim="$(arg is_sim)" x="0.25" y="0.0" z="0.33" topic="/imu/data"/>
+   <xacro:hunter_imu name="$(arg prefix)imu" is_sim="$(arg is_sim)" x="-0.25" y="0.0" z="0.47" topic="/gps_base/yaw"/>
+   <xacro:hunter_imu name="$(arg prefix)imu1" is_sim="$(arg is_sim)" x="0.25" y="0.0" z="0.47" topic="/imu/data"/>
    <!-- <xacro:hunter_lidar name="$(arg prefix)front_lidar" x="0.615" y="0.28" z="0.33" is_sim="$(arg is_sim)" /> -->
    <!-- <xacro:hunter_lidar name="$(arg prefix)back_lidar" x="-0.565" y="-0.28" z="0.33"  yaw="3.14" is_sim="$(arg is_sim)"/> -->
-   <xacro:hunter_depth_camera name="front_camera" x="0.55" y="-0.00" z="0.50" is_sim="$(arg is_sim)" />
-   <xacro:hunter_depth_camera name="back_camera" x="-0.55" y="-0.00" z="0.50" is_sim="$(arg is_sim)" yaw="3.14"/>
+   <xacro:hunter_depth_camera name="front_camera" x="0.55" y="-0.00" z="0.72" is_sim="$(arg is_sim)" />
+   <xacro:hunter_depth_camera name="back_camera" x="-0.55" y="-0.00" z="0.72" is_sim="$(arg is_sim)" yaw="3.14"/>
    <!-- <xacro:hunter_depth_camera name="fish_front_camera" x="0.55" y="0.00" z="0.93" is_sim="$(arg is_sim)" /> -->
    <!-- <xacro:hunter_depth_camera name="fish_right_camera" x="0.495" y="0.08" z="0.93" is_sim="$(arg is_sim)"  yaw="1.57"/> -->
    <!-- <xacro:hunter_depth_camera name="fish_back_camera" x="0.179" y="0.00" z="1.28" is_sim="$(arg is_sim)" yaw="3.14" />-->
    <!-- <xacro:hunter_depth_camera name="fish_left_camera" x="0.495" y="-0.08" z="0.93" is_sim="$(arg is_sim)" yaw="-1.57" /> -->
-   <xacro:hunter_gps name="$(arg prefix)gps_base" is_sim="$(arg is_sim)" x="-0.25" y="0.0" z="0.33" yaw="0.037482" />
+   <xacro:hunter_gps name="$(arg prefix)gps_base" is_sim="$(arg is_sim)" x="-0.25" y="0.0" z="0.47" yaw="0.037482" />
    <!-- <xacro:hunter_gps name="$(arg prefix)back_antenna" is_sim="$(arg is_sim)" x="-0.5" y="-0.245" z="0.80"/> -->
    <!-- <xacro:hunter_gps name="$(arg prefix)front_antenna" is_sim="$(arg is_sim)" x="0.5" y="-0.245" z="0.80"/> -->
-   <xacro:mid360 name="$(arg prefix)front_lidar_link" topic="front_lidar/points" origin_xyz="0.615 0.28 0.33" origin_rpy="${front_lidar_rpy}" is_sim="$(arg is_sim)"/>
-   <xacro:mid360 name="$(arg prefix)back_lidar_link" topic="back_lidar/points" origin_xyz="-0.615 -0.28 0.33" origin_rpy="${back_lidar_rpy}" is_sim="$(arg is_sim)"/>
+   <xacro:mid360 name="$(arg prefix)front_lidar_link" topic="front_lidar/points" origin_xyz="0.615 0.28 0.46" origin_rpy="${front_lidar_rpy}" is_sim="$(arg is_sim)"/>
+   <xacro:mid360 name="$(arg prefix)back_lidar_link" topic="back_lidar/points" origin_xyz="-0.615 -0.28 0.46" origin_rpy="${back_lidar_rpy}" is_sim="$(arg is_sim)"/>
 </robot>

Commit message: fine tune tf tree

File: hunter_pltf_description/description/hunter_pltf.urdf.xacro (robot description, xacro)
@@ -10,5 +10,5 @@
    <xacro:unless value="$(arg is_sim)">
       <xacro:include filename="$(find hunter_description)/description/robot_core_real_hack.xacro"/>
-      <xacro:property name="front_lidar_rpy" value="0 0 0"/>
+      <xacro:property name="front_lidar_rpy" value="-0.0174533 0 0"/>
       <xacro:property name="back_lidar_rpy" value="0 0 3.14159"/>
    </xacro:unless>
@@ -31,5 +31,5 @@
    <!-- <xacro:hunter_gps name="$(arg prefix)back_antenna" is_sim="$(arg is_sim)" x="-0.5" y="-0.245" z="0.80"/> -->
    <!-- <xacro:hunter_gps name="$(arg prefix)front_antenna" is_sim="$(arg is_sim)" x="0.5" y="-0.245" z="0.80"/> -->
-   <xacro:mid360 name="$(arg prefix)front_lidar_link" topic="front_lidar/points" origin_xyz="0.615 0.28 0.46" origin_rpy="${front_lidar_rpy}" is_sim="$(arg is_sim)"/>
-   <xacro:mid360 name="$(arg prefix)back_lidar_link" topic="back_lidar/points" origin_xyz="-0.615 -0.28 0.46" origin_rpy="${back_lidar_rpy}" is_sim="$(arg is_sim)"/>
+   <xacro:mid360 name="$(arg prefix)front_lidar_link" topic="front_lidar/points" origin_xyz="0.56 0.23 0.46" origin_rpy="${front_lidar_rpy}" is_sim="$(arg is_sim)"/>
+   <xacro:mid360 name="$(arg prefix)back_lidar_link" topic="back_lidar/points" origin_xyz="-0.56 -0.23 0.46" origin_rpy="${back_lidar_rpy}" is_sim="$(arg is_sim)"/>
 </robot>

Commit message: update urdf

File: hunter_pltf_description/description/hunter_pltf.urdf.xacro (robot description, xacro)
@@ -10,6 +10,6 @@
    <xacro:unless value="$(arg is_sim)">
       <xacro:include filename="$(find hunter_description)/description/robot_core_real_hack.xacro"/>
-      <xacro:property name="front_lidar_rpy" value="-0.0174533 0 0"/>
-      <xacro:property name="back_lidar_rpy" value="0 0 3.14159"/>
+      <xacro:property name="front_lidar_rpy" value="-0.0174533 0 0.00872665"/>
+      <xacro:property name="back_lidar_rpy" value="0 0 3.13286335"/>
    </xacro:unless>
    <xacro:include filename="$(find hunter_pltf_description)/description/lidar.urdf.xacro"/>
@@ -28,8 +28,8 @@
    <!-- <xacro:hunter_depth_camera name="fish_back_camera" x="0.179" y="0.00" z="1.28" is_sim="$(arg is_sim)" yaw="3.14" />-->
    <!-- <xacro:hunter_depth_camera name="fish_left_camera" x="0.495" y="-0.08" z="0.93" is_sim="$(arg is_sim)" yaw="-1.57" /> -->
-   <xacro:hunter_gps name="$(arg prefix)gps_base" is_sim="$(arg is_sim)" x="-0.25" y="0.0" z="0.47" yaw="0.037482" />
+   <xacro:hunter_gps name="$(arg prefix)gps_base" is_sim="$(arg is_sim)" x="-0.25" y="0.0" z="0.47" yaw="0.0" />
    <!-- <xacro:hunter_gps name="$(arg prefix)back_antenna" is_sim="$(arg is_sim)" x="-0.5" y="-0.245" z="0.80"/> -->
    <!-- <xacro:hunter_gps name="$(arg prefix)front_antenna" is_sim="$(arg is_sim)" x="0.5" y="-0.245" z="0.80"/> -->
-   <xacro:mid360 name="$(arg prefix)front_lidar_link" topic="front_lidar/points" origin_xyz="0.56 0.23 0.46" origin_rpy="${front_lidar_rpy}" is_sim="$(arg is_sim)"/>
-   <xacro:mid360 name="$(arg prefix)back_lidar_link" topic="back_lidar/points" origin_xyz="-0.56 -0.23 0.46" origin_rpy="${back_lidar_rpy}" is_sim="$(arg is_sim)"/>
+   <xacro:mid360 name="$(arg prefix)front_lidar_link" topic="front_lidar/points" origin_xyz="0.56 0.235 0.46" origin_rpy="${front_lidar_rpy}" is_sim="$(arg is_sim)"/>
+   <xacro:mid360 name="$(arg prefix)back_lidar_link" topic="back_lidar/points" origin_xyz="-0.56 -0.235 0.46" origin_rpy="${back_lidar_rpy}" is_sim="$(arg is_sim)"/>
 </robot>

Commit message: update with main  (#24)
* Update lidar properties and adjust downsample rate in mid360 configuration

* Update IMU configuration in hunter_pltf.urdf.xacro

* fix urdf

* fine tune tf tree

* update urdf

* Dependency to ros2_livox_simulation package added (#23)

---------

Co-authored-by: A. Yilmaz <79148268+yilmazabdurrah@users.noreply.github.com>

File: hunter_pltf_description/description/hunter_pltf.urdf.xacro (robot description, xacro)
@@ -5,7 +5,11 @@
    <xacro:if value="$(arg is_sim)">
       <xacro:include filename="$(find hunter_description)/description/robot.urdf.xacro"/>
+      <xacro:property name="front_lidar_rpy" value="0 0 0"/>
+      <xacro:property name="back_lidar_rpy" value="0 0 3.14159"/>
    </xacro:if>
    <xacro:unless value="$(arg is_sim)">
-   <xacro:include filename="$(find hunter_description)/description/robot_core_real_hack.xacro"/>
+      <xacro:include filename="$(find hunter_description)/description/robot_core_real_hack.xacro"/>
+      <xacro:property name="front_lidar_rpy" value="-0.0174533 0 0.00872665"/>
+      <xacro:property name="back_lidar_rpy" value="0 0 3.13286335"/>
    </xacro:unless>
    <xacro:include filename="$(find hunter_pltf_description)/description/lidar.urdf.xacro"/>
@@ -14,17 +18,18 @@
    <xacro:include filename="$(find hunter_pltf_description)/description/gps.urdf.xacro"/>
    <xacro:include filename="$(find hunter_pltf_description)/description/depth_camera.urdf.xacro"/>
-   <xacro:hunter_imu name="$(arg prefix)imu1" is_sim="$(arg is_sim)" x="0.0" y="0.0" z="0.2" topic="/gps_base/yaw"/>
+   <xacro:hunter_imu name="$(arg prefix)imu" is_sim="$(arg is_sim)" x="-0.25" y="0.0" z="0.47" topic="/gps_base/yaw"/>
+   <xacro:hunter_imu name="$(arg prefix)imu1" is_sim="$(arg is_sim)" x="0.25" y="0.0" z="0.47" topic="/imu/data"/>
    <!-- <xacro:hunter_lidar name="$(arg prefix)front_lidar" x="0.615" y="0.28" z="0.33" is_sim="$(arg is_sim)" /> -->
    <!-- <xacro:hunter_lidar name="$(arg prefix)back_lidar" x="-0.565" y="-0.28" z="0.33"  yaw="3.14" is_sim="$(arg is_sim)"/> -->
-   <xacro:hunter_depth_camera name="front_camera" x="0.55" y="-0.00" z="0.50" is_sim="$(arg is_sim)" />
-   <xacro:hunter_depth_camera name="back_camera" x="-0.55" y="-0.00" z="0.50" is_sim="$(arg is_sim)" yaw="3.14"/>
+   <xacro:hunter_depth_camera name="front_camera" x="0.55" y="-0.00" z="0.72" is_sim="$(arg is_sim)" />
+   <xacro:hunter_depth_camera name="back_camera" x="-0.55" y="-0.00" z="0.72" is_sim="$(arg is_sim)" yaw="3.14"/>
    <!-- <xacro:hunter_depth_camera name="fish_front_camera" x="0.55" y="0.00" z="0.93" is_sim="$(arg is_sim)" /> -->
    <!-- <xacro:hunter_depth_camera name="fish_right_camera" x="0.495" y="0.08" z="0.93" is_sim="$(arg is_sim)"  yaw="1.57"/> -->
    <!-- <xacro:hunter_depth_camera name="fish_back_camera" x="0.179" y="0.00" z="1.28" is_sim="$(arg is_sim)" yaw="3.14" />-->
    <!-- <xacro:hunter_depth_camera name="fish_left_camera" x="0.495" y="-0.08" z="0.93" is_sim="$(arg is_sim)" yaw="-1.57" /> -->
-   <xacro:hunter_gps name="$(arg prefix)gps_base" is_sim="$(arg is_sim)" x="-0.25" y="0.0" z="0.33" yaw="0.037482" />
+   <xacro:hunter_gps name="$(arg prefix)gps_base" is_sim="$(arg is_sim)" x="-0.25" y="0.0" z="0.47" yaw="0.0" />
    <!-- <xacro:hunter_gps name="$(arg prefix)back_antenna" is_sim="$(arg is_sim)" x="-0.5" y="-0.245" z="0.80"/> -->
    <!-- <xacro:hunter_gps name="$(arg prefix)front_antenna" is_sim="$(arg is_sim)" x="0.5" y="-0.245" z="0.80"/> -->
-   <xacro:mid360 name="$(arg prefix)front_lidar_link" topic="front_lidar/points" origin_xyz="0.615 0.28 0.33" origin_rpy="0 0 -0.0261799" is_sim="$(arg is_sim)"/>
-   <xacro:mid360 name="$(arg prefix)back_lidar_link" topic="back_lidar/points" origin_xyz="-0.615 -0.28 0.33" origin_rpy="-0.174533 0 3.14159" is_sim="$(arg is_sim)"/>
+   <xacro:mid360 name="$(arg prefix)front_lidar_link" topic="front_lidar/points" origin_xyz="0.56 0.235 0.46" origin_rpy="${front_lidar_rpy}" is_sim="$(arg is_sim)"/>
+   <xacro:mid360 name="$(arg prefix)back_lidar_link" topic="back_lidar/points" origin_xyz="-0.56 -0.235 0.46" origin_rpy="${back_lidar_rpy}" is_sim="$(arg is_sim)"/>
 </robot>
