Commit message: Implement YAML-based robot configuration system
- Add config/robots directory with default.yaml and hunter_01.yaml
- Create config_loader.py for loading and merging configurations
- Update hunter_pltf.urdf.xacro to accept sensor pose parameters
- Modify launch files (pltf_rsp, bringup, gazebo) to use robot_id arg
- Add comprehensive README.md with usage documentation
- Enable per-robot sensor calibration without separate xacro files

Co-authored-by: marc-hanheide <1153084+marc-hanheide@users.noreply.github.com>

File: hunter_pltf_description/description/hunter_pltf.urdf.xacro (robot description, xacro)
@@ -3,13 +3,69 @@
    <xacro:arg name="is_sim" default="true"/>
    <xacro:arg name="prefix" default="" />
+   <!-- IMU sensor parameters -->
+   <xacro:arg name="imu_x" default="-0.25"/>
+   <xacro:arg name="imu_y" default="0.0"/>
+   <xacro:arg name="imu_z" default="0.47"/>
+   <xacro:arg name="imu_roll" default="0.0"/>
+   <xacro:arg name="imu_pitch" default="0.0"/>
+   <xacro:arg name="imu_yaw" default="0.0"/>
+   <xacro:arg name="imu_topic" default="/gps_base/yaw"/>
+   <xacro:arg name="imu1_x" default="0.25"/>
+   <xacro:arg name="imu1_y" default="0.0"/>
+   <xacro:arg name="imu1_z" default="0.47"/>
+   <xacro:arg name="imu1_roll" default="0.0"/>
+   <xacro:arg name="imu1_pitch" default="0.0"/>
+   <xacro:arg name="imu1_yaw" default="0.0"/>
+   <xacro:arg name="imu1_topic" default="/imu/data"/>
+   <!-- Camera parameters -->
+   <xacro:arg name="front_camera_x" default="0.55"/>
+   <xacro:arg name="front_camera_y" default="0.0"/>
+   <xacro:arg name="front_camera_z" default="0.72"/>
+   <xacro:arg name="front_camera_roll" default="0.0"/>
+   <xacro:arg name="front_camera_pitch" default="0.0"/>
+   <xacro:arg name="front_camera_yaw" default="0.0"/>
+   <xacro:arg name="back_camera_x" default="-0.55"/>
+   <xacro:arg name="back_camera_y" default="0.0"/>
+   <xacro:arg name="back_camera_z" default="0.72"/>
+   <xacro:arg name="back_camera_roll" default="0.0"/>
+   <xacro:arg name="back_camera_pitch" default="0.0"/>
+   <xacro:arg name="back_camera_yaw" default="3.14159265359"/>
+   <!-- GPS parameters -->
+   <xacro:arg name="gps_base_x" default="-0.25"/>
+   <xacro:arg name="gps_base_y" default="0.0"/>
+   <xacro:arg name="gps_base_z" default="0.47"/>
+   <xacro:arg name="gps_base_roll" default="0.0"/>
+   <xacro:arg name="gps_base_pitch" default="0.0"/>
+   <xacro:arg name="gps_base_yaw" default="0.0"/>
+   <!-- LiDAR parameters -->
+   <xacro:arg name="front_lidar_x" default="0.56"/>
+   <xacro:arg name="front_lidar_y" default="0.235"/>
+   <xacro:arg name="front_lidar_z" default="0.46"/>
+   <xacro:arg name="front_lidar_roll_sim" default="0.0"/>
+   <xacro:arg name="front_lidar_pitch_sim" default="0.0"/>
+   <xacro:arg name="front_lidar_yaw_sim" default="0.0"/>
+   <xacro:arg name="front_lidar_roll_real" default="-0.0174533"/>
+   <xacro:arg name="front_lidar_pitch_real" default="0.0"/>
+   <xacro:arg name="front_lidar_yaw_real" default="0.00872665"/>
+   <xacro:arg name="front_lidar_topic" default="front_lidar/points"/>
+   <xacro:arg name="back_lidar_x" default="-0.56"/>
+   <xacro:arg name="back_lidar_y" default="-0.235"/>
+   <xacro:arg name="back_lidar_z" default="0.46"/>
+   <xacro:arg name="back_lidar_roll_sim" default="0.0"/>
+   <xacro:arg name="back_lidar_pitch_sim" default="0.0"/>
+   <xacro:arg name="back_lidar_yaw_sim" default="3.14159265359"/>
+   <xacro:arg name="back_lidar_roll_real" default="0.0"/>
+   <xacro:arg name="back_lidar_pitch_real" default="0.0"/>
+   <xacro:arg name="back_lidar_yaw_real" default="3.13286335"/>
+   <xacro:arg name="back_lidar_topic" default="back_lidar/points"/>
    <xacro:if value="$(arg is_sim)">
       <xacro:include filename="$(find hunter_description)/description/robot.urdf.xacro"/>
-      <xacro:property name="front_lidar_rpy" value="0 0 0"/>
-      <xacro:property name="back_lidar_rpy" value="0 0 3.14159"/>
+      <xacro:property name="front_lidar_rpy" value="$(arg front_lidar_roll_sim) $(arg front_lidar_pitch_sim) $(arg front_lidar_yaw_sim)"/>
+      <xacro:property name="back_lidar_rpy" value="$(arg back_lidar_roll_sim) $(arg back_lidar_pitch_sim) $(arg back_lidar_yaw_sim)"/>
    </xacro:if>
    <xacro:unless value="$(arg is_sim)">
       <xacro:include filename="$(find hunter_description)/description/robot_core_real_hack.xacro"/>
-      <xacro:property name="front_lidar_rpy" value="-0.0174533 0 0.00872665"/>
-      <xacro:property name="back_lidar_rpy" value="0 0 3.13286335"/>
+      <xacro:property name="front_lidar_rpy" value="$(arg front_lidar_roll_real) $(arg front_lidar_pitch_real) $(arg front_lidar_yaw_real)"/>
+      <xacro:property name="back_lidar_rpy" value="$(arg back_lidar_roll_real) $(arg back_lidar_pitch_real) $(arg back_lidar_yaw_real)"/>
    </xacro:unless>
    <xacro:include filename="$(find hunter_pltf_description)/description/lidar.urdf.xacro"/>
@@ -18,18 +74,36 @@
    <xacro:include filename="$(find hunter_pltf_description)/description/gps.urdf.xacro"/>
    <xacro:include filename="$(find hunter_pltf_description)/description/depth_camera.urdf.xacro"/>
-   <xacro:hunter_imu name="$(arg prefix)imu" is_sim="$(arg is_sim)" x="-0.25" y="0.0" z="0.47" topic="/gps_base/yaw"/>
-   <xacro:hunter_imu name="$(arg prefix)imu1" is_sim="$(arg is_sim)" x="0.25" y="0.0" z="0.47" topic="/imu/data"/>
+   <xacro:hunter_imu name="$(arg prefix)imu" is_sim="$(arg is_sim)"
+                     x="$(arg imu_x)" y="$(arg imu_y)" z="$(arg imu_z)"
+                     roll="$(arg imu_roll)" pitch="$(arg imu_pitch)" yaw="$(arg imu_yaw)"
+                     topic="$(arg imu_topic)"/>
+   <xacro:hunter_imu name="$(arg prefix)imu1" is_sim="$(arg is_sim)"
+                     x="$(arg imu1_x)" y="$(arg imu1_y)" z="$(arg imu1_z)"
+                     roll="$(arg imu1_roll)" pitch="$(arg imu1_pitch)" yaw="$(arg imu1_yaw)"
+                     topic="$(arg imu1_topic)"/>
    <!-- <xacro:hunter_lidar name="$(arg prefix)front_lidar" x="0.615" y="0.28" z="0.33" is_sim="$(arg is_sim)" /> -->
    <!-- <xacro:hunter_lidar name="$(arg prefix)back_lidar" x="-0.565" y="-0.28" z="0.33"  yaw="3.14" is_sim="$(arg is_sim)"/> -->
-   <xacro:hunter_depth_camera name="front_camera" x="0.55" y="-0.00" z="0.72" is_sim="$(arg is_sim)" />
-   <xacro:hunter_depth_camera name="back_camera" x="-0.55" y="-0.00" z="0.72" is_sim="$(arg is_sim)" yaw="3.14"/>
+   <xacro:hunter_depth_camera name="front_camera"
+                              x="$(arg front_camera_x)" y="$(arg front_camera_y)" z="$(arg front_camera_z)"
+                              roll="$(arg front_camera_roll)" pitch="$(arg front_camera_pitch)" yaw="$(arg front_camera_yaw)"
+                              is_sim="$(arg is_sim)" />
+   <xacro:hunter_depth_camera name="back_camera"
+                              x="$(arg back_camera_x)" y="$(arg back_camera_y)" z="$(arg back_camera_z)"
+                              roll="$(arg back_camera_roll)" pitch="$(arg back_camera_pitch)" yaw="$(arg back_camera_yaw)"
+                              is_sim="$(arg is_sim)"/>
    <!-- <xacro:hunter_depth_camera name="fish_front_camera" x="0.55" y="0.00" z="0.93" is_sim="$(arg is_sim)" /> -->
    <!-- <xacro:hunter_depth_camera name="fish_right_camera" x="0.495" y="0.08" z="0.93" is_sim="$(arg is_sim)"  yaw="1.57"/> -->
    <!-- <xacro:hunter_depth_camera name="fish_back_camera" x="0.179" y="0.00" z="1.28" is_sim="$(arg is_sim)" yaw="3.14" />-->
    <!-- <xacro:hunter_depth_camera name="fish_left_camera" x="0.495" y="-0.08" z="0.93" is_sim="$(arg is_sim)" yaw="-1.57" /> -->
-   <xacro:hunter_gps name="$(arg prefix)gps_base" is_sim="$(arg is_sim)" x="-0.25" y="0.0" z="0.47" yaw="0.0" />
+   <xacro:hunter_gps name="$(arg prefix)gps_base" is_sim="$(arg is_sim)"
+                     x="$(arg gps_base_x)" y="$(arg gps_base_y)" z="$(arg gps_base_z)"
+                     roll="$(arg gps_base_roll)" pitch="$(arg gps_base_pitch)" yaw="$(arg gps_base_yaw)" />
    <!-- <xacro:hunter_gps name="$(arg prefix)back_antenna" is_sim="$(arg is_sim)" x="-0.5" y="-0.245" z="0.80"/> -->
    <!-- <xacro:hunter_gps name="$(arg prefix)front_antenna" is_sim="$(arg is_sim)" x="0.5" y="-0.245" z="0.80"/> -->
-   <xacro:mid360 name="$(arg prefix)front_lidar_link" topic="front_lidar/points" origin_xyz="0.56 0.235 0.46" origin_rpy="${front_lidar_rpy}" is_sim="$(arg is_sim)"/>
-   <xacro:mid360 name="$(arg prefix)back_lidar_link" topic="back_lidar/points" origin_xyz="-0.56 -0.235 0.46" origin_rpy="${back_lidar_rpy}" is_sim="$(arg is_sim)"/>
+   <xacro:mid360 name="$(arg prefix)front_lidar_link" topic="$(arg front_lidar_topic)"
+                 origin_xyz="$(arg front_lidar_x) $(arg front_lidar_y) $(arg front_lidar_z)"
+                 origin_rpy="${front_lidar_rpy}" is_sim="$(arg is_sim)"/>
+   <xacro:mid360 name="$(arg prefix)back_lidar_link" topic="$(arg back_lidar_topic)"
+                 origin_xyz="$(arg back_lidar_x) $(arg back_lidar_y) $(arg back_lidar_z)"
+                 origin_rpy="${back_lidar_rpy}" is_sim="$(arg is_sim)"/>
 </robot>

Commit message: Refactor launch and URDF files to integrate Mid-360 LiDAR support and enhance simulation parameters

File: hunter_pltf_description/description/hunter_pltf.urdf.xacro (robot description, xacro)
@@ -13,25 +13,35 @@
       <xacro:property name="back_lidar_rpy" value="0 0 3.13286335"/>
    </xacro:unless>
-   <!--
-     MIGRATION: replaced the Gazebo-Classic Livox includes
-     (lidar.urdf.xacro, mid360.xacro) with a single vendor-neutral 3D LiDAR
-     macro (lidar_3d.urdf.xacro) that uses the native gz-sim `gpu_lidar` sensor.
-   -->
-   <xacro:include filename="$(find hunter_pltf_description)/description/lidar_3d.urdf.xacro"/>
+   <xacro:include filename="$(find hunter_pltf_description)/description/mid360_lidar.urdf.xacro"/>
    <xacro:include filename="$(find hunter_pltf_description)/description/imu.urdf.xacro"/>
    <xacro:include filename="$(find hunter_pltf_description)/description/gps.urdf.xacro"/>
    <xacro:include filename="$(find hunter_pltf_description)/description/depth_camera.urdf.xacro"/>
    <xacro:hunter_imu name="$(arg prefix)imu" is_sim="$(arg is_sim)" x="-0.25" y="0.0" z="0.47" topic="/gps_base/yaw"/>
-   <xacro:hunter_imu name="$(arg prefix)imu1" is_sim="$(arg is_sim)" x="0.25" y="0.0" z="0.47" topic="/imu/data"/>
    <xacro:hunter_depth_camera name="front_camera" x="0.55" y="-0.00" z="0.72" is_sim="$(arg is_sim)" />
    <xacro:hunter_depth_camera name="back_camera" x="-0.55" y="-0.00" z="0.72" is_sim="$(arg is_sim)" yaw="3.14"/>
    <xacro:hunter_gps name="$(arg prefix)gps_base" is_sim="$(arg is_sim)" x="-0.25" y="0.0" z="0.47" yaw="0.0" />
-   <!--
-     3D LiDARs. The `gpu_lidar` sensor publishes the point cloud on
-     "<topic>/points", so we pass the base topic name here (e.g. "front_lidar")
-     and the cloud appears on "front_lidar/points" - same topic the rest of the
-     stack previously expected from the Livox plugin.
-   -->
-   <xacro:lidar_3d name="$(arg prefix)front_lidar_link" topic="front_lidar" origin_xyz="0.56 0.235 0.46" origin_rpy="${front_lidar_rpy}" is_sim="$(arg is_sim)"/>
-   <xacro:lidar_3d name="$(arg prefix)back_lidar_link" topic="back_lidar" origin_xyz="-0.56 -0.235 0.46" origin_rpy="${back_lidar_rpy}" is_sim="$(arg is_sim)"/>
+   <xacro:mid360_lidar name="$(arg prefix)front_lidar_link"
+                       frame_id="$(arg prefix)front_lidar_link"
+                       raw_topic="front_lidar/raw_gpu"
+                       points_topic="front_lidar/points"
+                       diagnostics_topic="front_lidar/diagnostics"
+                       origin_xyz="0.56 0.235 0.46"
+                       origin_rpy="${front_lidar_rpy}"
+                       is_sim="$(arg is_sim)"/>
+   <xacro:hunter_imu name="$(arg prefix)front_lidar_imu"
+                     parent="$(arg prefix)front_lidar_link"
+                     is_sim="$(arg is_sim)"
+                     x="0.0" y="0.0" z="-0.047"
+                     topic="front_lidar/imu"
+                     update_rate="200"
+                     angular_velocity_stddev="0.005"
+                     linear_acceleration_stddev="0.02"/>
+   <xacro:mid360_lidar name="$(arg prefix)back_lidar_link"
+                       frame_id="$(arg prefix)back_lidar_link"
+                       raw_topic="back_lidar/raw_gpu"
+                       points_topic="back_lidar/points"
+                       diagnostics_topic="back_lidar/diagnostics"
+                       origin_xyz="-0.56 -0.235 0.46"
+                       origin_rpy="${back_lidar_rpy}"
+                       is_sim="$(arg is_sim)"/>
 </robot>

File: hunter_pltf_description/description/imu.urdf.xacro (robot description, xacro)
@@ -1,7 +1,14 @@
 <?xml version="1.0"?>
 <robot xmlns:xacro="http://www.ros.org/wiki/xacro">
-  <xacro:macro name="hunter_imu" params="name topic x:=0.0 y:=0.0 z:=0.0 roll:=0.0 pitch:=0.0 yaw:=0.0 is_sim:=true">
+  <xacro:macro name="hunter_imu"
+               params="name topic parent:=base_link
+                       x:=0.0 y:=0.0 z:=0.0 roll:=0.0 pitch:=0.0 yaw:=0.0
+                       update_rate:=50
+                       angular_velocity_stddev:=0.01
+                       linear_acceleration_stddev:=0.01
+                       bias_stddev:=0.0001
+                       is_sim:=true">
     <joint name="${name}_joint" type="fixed">
-      <parent link="base_link"/>
+      <parent link="${parent}"/>
       <child link="${name}_link"/>
       <origin xyz="${x} ${y} ${z}" rpy="${roll} ${pitch} ${yaw}"/>
@@ -13,5 +20,5 @@
           <topic>${topic}</topic>
           <always_on>true</always_on>
-          <update_rate>50</update_rate>
+          <update_rate>${update_rate}</update_rate>
           <imu>
             <angular_velocity>
@@ -19,7 +26,7 @@
                 <noise type="gaussian">
                   <mean>0.0</mean>
-                  <stddev>0.01</stddev>
+                  <stddev>${angular_velocity_stddev}</stddev>
                   <bias_mean>0.0</bias_mean>
-                  <bias_stddev>0.0001</bias_stddev>
+                  <bias_stddev>${bias_stddev}</bias_stddev>
                 </noise>
               </x>
@@ -27,7 +34,7 @@
                 <noise type="gaussian">
                   <mean>0.0</mean>
-                  <stddev>0.01</stddev>
+                  <stddev>${angular_velocity_stddev}</stddev>
                   <bias_mean>0.0</bias_mean>
-                  <bias_stddev>0.0001</bias_stddev>
+                  <bias_stddev>${bias_stddev}</bias_stddev>
                 </noise>
               </y>
@@ -35,7 +42,7 @@
                 <noise type="gaussian">
                   <mean>0.0</mean>
-                  <stddev>0.01</stddev>
+                  <stddev>${angular_velocity_stddev}</stddev>
                   <bias_mean>0.0</bias_mean>
-                  <bias_stddev>0.0001</bias_stddev>
+                  <bias_stddev>${bias_stddev}</bias_stddev>
                 </noise>
               </z>
@@ -45,7 +52,7 @@
                 <noise type="gaussian">
                   <mean>0.0</mean>
-                  <stddev>0.01</stddev>
+                  <stddev>${linear_acceleration_stddev}</stddev>
                   <bias_mean>0.0</bias_mean>
-                  <bias_stddev>0.0001</bias_stddev>
+                  <bias_stddev>${bias_stddev}</bias_stddev>
                 </noise>
               </x>
@@ -53,7 +60,7 @@
                 <noise type="gaussian">
                   <mean>0.0</mean>
-                  <stddev>0.01</stddev>
+                  <stddev>${linear_acceleration_stddev}</stddev>
                   <bias_mean>0.0</bias_mean>
-                  <bias_stddev>0.0001</bias_stddev>
+                  <bias_stddev>${bias_stddev}</bias_stddev>
                 </noise>
               </y>
@@ -61,7 +68,7 @@
                 <noise type="gaussian">
                   <mean>0.0</mean>
-                  <stddev>0.01</stddev>
+                  <stddev>${linear_acceleration_stddev}</stddev>
                   <bias_mean>0.0</bias_mean>
-                  <bias_stddev>0.0001</bias_stddev>
+                  <bias_stddev>${bias_stddev}</bias_stddev>
                 </noise>
               </z>
