Commit message: Enhance IMU and mid360 configurations by adding new parameters for flexibility and improved sensor properties

File: hunter_pltf_description/description/imu.urdf.xacro (robot description, xacro)
@@ -1,9 +1,10 @@
 <?xml version="1.0"?>
 <robot xmlns:xacro="http://www.ros.org/wiki/xacro">
-  <xacro:macro name="hunter_imu" params="name topic x:=0.0 y:=0.0 z:=0.0 roll:=0.0 pitch:=0.0 yaw:=0.0 is_sim:=true">
+  <xacro:macro name="hunter_imu" params="name topic parent:=base_link x:=0.0 y:=0.0 z:=0.0 roll:=0.0 pitch:=0.0 yaw:=0.0 rpy:='' is_sim:=true update_rate:=50 angular_velocity_stddev:=0.01 linear_acceleration_stddev:=0.01">
+    <xacro:property name="origin_rpy" value="${rpy if rpy else str(roll) + ' ' + str(pitch) + ' ' + str(yaw)}"/>
     <joint name="${name}_joint" type="fixed">
-      <parent link="base_link"/>
+      <parent link="${parent}"/>
       <child link="${name}_link"/>
-      <origin xyz="${x} ${y} ${z}" rpy="${roll} ${pitch} ${yaw}"/>
+      <origin xyz="${x} ${y} ${z}" rpy="${origin_rpy}"/>
     </joint>
     <link name="${name}_link"/>
@@ -19,10 +20,10 @@
           </plugin>
           <always_on>true</always_on>
-          <update_rate>50</update_rate>
+          <update_rate>${update_rate}</update_rate>
           <imu>
             <angular_velocity>
               <noise type="gaussian">
                 <mean>0.0</mean>
-                <stddev>0.01</stddev>
+                <stddev>${angular_velocity_stddev}</stddev>
               </noise>
               <bias>
@@ -34,5 +35,5 @@
               <noise type="gaussian">
                 <mean>0.0</mean>
-                <stddev>0.01</stddev>
+                <stddev>${linear_acceleration_stddev}</stddev>
               </noise>
               <bias>

File: hunter_pltf_description/description/mid360.xacro (robot description, xacro)
@@ -30,8 +30,10 @@
                        raw_topic:='mid360/raw_gpu'
                        topic:='mid360/points'
+                       points_topic:=''
                        diagnostics_topic:='mid360/diagnostics'
                        frame_id:=''
                        origin_xyz='0 0 0' origin_rpy='0 0 0'
                        is_sim:=true">
+              <xacro:property name="resolved_topic" value="${points_topic if points_topic else topic}"/>
     <link name="${name}">
       <xacro:box_inertia m="${mass}" w="${width}" d="${length}" h="${height}"/>
@@ -87,5 +89,5 @@
                 name="livox_mid360_gz::LivoxMid360GpuLidar">
           <input_topic>${raw_topic}/points</input_topic>
-          <output_topic>${topic}</output_topic>
+          <output_topic>${resolved_topic}</output_topic>
           <diagnostics_topic>${diagnostics_topic}</diagnostics_topic>
           <frame_id>${frame_id}</frame_id>
